File: hardware/interposer/interposer.kicad_pcb (KiCad board)
At the start: 2 copper layers, 64.5 x 95.5 mm, 9 parts, among them J1 Conn_02x16_Odd_Even, J2 DNF, J3 DNF

Commit message: updated interposer
Parts:
- moved G*** 2.58 mm to (97.5, 37.5)
Routing:
- net GND: vias 17 -> 23
Other:
- outline, holes or cut-outs redrawn
Changed lines of the file:
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@@
       (layerselection 0x00010fc_ffffffff)
       (disableapertmacros false)
-      (usegerberextensions false)
+      (usegerberextensions true)
       (usegerberattributes false)
       (usegerberadvancedattributes false)
-      (creategerberjobfile true)
+      (creategerberjobfile false)
       (svguseinch false)
       (svgprecision 6)
-      (excludeedgelayer false)
+      (excludeedgelayer true)
       (plotframeref false)
       (viasonmask false)
@@
       (psa4output false)
       (plotreference true)
-      (plotvalue true)
+      (plotvalue false)
       (plotinvisibletext false)
       (sketchpadsonfab false)
-      (subtractmaskfromsilk false)
+      (subtractmaskfromsilk true)
       (outputformat 1)
       (mirror false)
@@
   )
   (footprint "interposer:loona" (layer "B.Cu")
-    (at 99.89 38.48 180)
+    (at 97.5 37.5 180)
     (attr board_only exclude_from_pos_files exclude_from_bom)
     (fp_text reference "G***" (at -7.95 -15.51) (layer "B.SilkS")
@@
   (gr_line (start 74.3 91.4) (end 74.3 39) (layer "Edge.Cuts") (width 0.15))
   (gr_line (start 67.25 4.5) (end 82.25 4.5) (layer "Edge.Cuts") (width 0.15))
-  (gr_line (start 121.7 39) (end 121.75 38.75) (layer "Edge.Cuts") (width 0.15))
-  (gr_line (start 121.75 38.75) (end 121.75 37.5) (layer "Edge.Cuts") (width 0.15))
+  (gr_line (start 122 25) (end 131.75 24.25) (layer "Edge.Cuts") (width 0.15))
+  (gr_line (start 74.3 39) (end 74 25) (layer "Edge.Cuts") (width 0.15))
+  (gr_line (start 74 25) (end 67.25 24.5) (layer "Edge.Cuts") (width 0.15))
   (gr_line (start 125.7 91.4) (end 125.7 41.6) (layer "Edge.Cuts") (width 0.15))
   (gr_line (start 75.4 100) (end 124.6 100) (layer "Edge.Cuts") (width 0.15))
   (gr_line (start 131.75 4.5) (end 131.25 4.5) (layer "Edge.Cuts") (width 0.15))
   (gr_line (start 131.75 24.25) (end 131.75 9.5) (layer "Edge.Cuts") (width 0.15))
-  (gr_line (start 125.75 37.5) (end 131.75 24.25) (layer "Edge.Cuts") (width 0.15))
   (gr_line (start 124.6 100) (end 124.6 91.4) (layer "Edge.Cuts") (width 0.15))
   (gr_line (start 121.7 39) (end 121.7 41.6) (layer "Edge.Cuts") (width 0.15))
   (gr_line (start 124.6 91.4) (end 125.7 91.4) (layer "Edge.Cuts") (width 0.15))
-  (gr_line (start 121.75 37.5) (end 125.75 37.5) (layer "Edge.Cuts") (width 0.15))
   (gr_line (start 125.7 41.6) (end 121.7 41.6) (layer "Edge.Cuts") (width 0.15))
   (gr_line (start 67.25 24.5) (end 67.25 4.5) (layer "Edge.Cuts") (width 0.15))
@@
   (gr_line (start 75.4 100) (end 75.4 91.4) (layer "Edge.Cuts") (width 0.15))
   (gr_line (start 131.75 9.5) (end 131.75 4.5) (layer "Edge.Cuts") (width 0.15))
-  (gr_line (start 74.3 39) (end 67.25 24.5) (layer "Edge.Cuts") (width 0.15))
   (gr_line (start 82.25 4.5) (end 131.25 4.5) (layer "Edge.Cuts") (width 0.15))
+  (gr_line (start 121.7 39) (end 122 25) (layer "Edge.Cuts") (width 0.15))
   (gr_text "whatever,\nloser" (at 100.08 69.53) (layer "B.SilkS")
     (effects (font (size 1.5 1.5) (thickness 0.3)) (justify mirror))
@@
   (via (at 99.23 64.02) (size 0.6) (drill 0.4) (layers "F.Cu" "B.Cu") (free) (net 2))
   (via (at 123.9 84) (size 1) (drill 0.8) (layers "F.Cu" "B.Cu") (net 2))
+  (via (at 78.486 55.626) (size 0.6) (drill 0.4) (layers "F.Cu" "B.Cu") (free) (net 2))
+  (via (at 99.06 90.17) (size 0.6) (drill 0.4) (layers "F.Cu" "B.Cu") (free) (net 2))
+  (via (at 78.486 76.962) (size 0.6) (drill 0.4) (layers "F.Cu" "B.Cu") (free) (net 2))
   (via (at 123.4 90.2) (size 1) (drill 0.8) (layers "F.Cu" "B.Cu") (net 2))
   (via (at 123.4 92.6) (size 0.6) (drill 0.4) (layers "F.Cu" "B.Cu") (net 2))
   (via (at 95.27 35.3) (size 0.6) (drill 0.4) (layers "F.Cu" "B.Cu") (free) (net 2))
+  (via (at 76.2 47.498) (size 0.6) (drill 0.4) (layers "F.Cu" "B.Cu") (free) (net 2))
+  (via (at 78.486 85.344) (size 0.6) (drill 0.4) (layers "F.Cu" "B.Cu") (free) (net 2))
   (via (at 120.7 68.5) (size 1) (drill 0.8) (layers "F.Cu" "B.Cu") (net 2))
   (via (at 87.17 34.19) (size 0.6) (drill 0.4) (layers "F.Cu" "B.Cu") (free) (net 2))
+  (via (at 78.486 66.548) (size 0.6) (drill 0.4) (layers "F.Cu" "B.Cu") (free) (net 2))
   (segment (start 77.7 44.3) (end 77.8 44.4) (width 0.4) (layer "F.Cu") (net 3))
   (segment (start 77.8 42.1) (end 77.7 42) (width 0.4) (layer "F.Cu") (net 3))
