File: hardware/gbpunk/gbpunk.kicad_sch (KiCad schematic)
At the start: 59 parts, among them J1 CART, J2 SWD_CONNECTOR, J4 SWD_CONNECTOR, P1 USB_C_CONNECTOR, SW7 RESET, SW9 USB_BOOT, U1 RP2040, U2 SN74LVC4245A, U3 W25Q128JVS, U4 NCP1117-3.3_SOT223, U5 SN74LVC4245A, U6 SN74LVC4245A, U7 SN74LVC4245A, Y1 12MHz

Commit message: need to double check but hardware rev looks good
Parts:
- removed C7: 27pF, Capacitor_SMD:C_0402_1005Metric_Pad0.74x0.62mm_HandSolder, symbol Device:C_Small
- removed J2: SWD_CONNECTOR, Connector_PinHeader_2.54mm:PinHeader_1x05_P2.54mm_Vertical, symbol Connector_Generic:Conn_01x05
- removed J4: SWD_CONNECTOR, Connector_PinHeader_1.27mm:PinHeader_2x05_P1.27mm_Vertical_SMD, symbol Connector:Conn_ARM_JTAG_SWD_10
- removed JP1, JP3, JP4: SWDIR_1, Jumper:SolderJumper-3_P1.3mm_Bridged12_RoundedPad1.0x1.5mm, symbol Jumper:Jumper_3_Bridged12
- removed JP2: SWDIR_0, Jumper:SolderJumper-3_P1.3mm_Bridged12_RoundedPad1.0x1.5mm, symbol Jumper:Jumper_3_Bridged12
- removed P1: USB_C_CONNECTOR, Connector_USB:USB_C_Receptacle_HRO_TYPE-C-31-M-12, symbol Connector:USB_C_Plug
- removed R10: 1k, Resistor_SMD:R_0402_1005Metric_Pad0.72x0.64mm_HandSolder, symbol Device:R
- removed R2, R3, R4, R5, R6, R7: 1k, Resistor_SMD:R_0603_1608Metric_Pad0.98x0.95mm_HandSolder, symbol Device:R
- removed TP2: RUN_TP, TestPoint:TestPoint_Pad_D1.0mm, symbol Connector:TestPoint
- removed TP4: DBUS_DIR_TP, TestPoint:TestPoint_Pad_D1.0mm, symbol Connector:TestPoint
- removed U1: RP2040, gbpunk:RP2040-QFN-56, symbol gbpunk:RP2040
- removed Y1: 12MHz, Crystal:Crystal_HC52-8mm_Vertical, symbol Device:Crystal_Small
- added C1, C2, C3: 4.7uF, Capacitor_SMD:C_0805_2012Metric, symbol Device:C_Small
- added C21: 100nF, Capacitor_SMD:C_0402_1005Metric, symbol Device:C_Small
- added C22, C23, C24, C26, C27: 10uF, Capacitor_SMD:C_0603_1608Metric_Pad1.08x0.95mm_HandSolder, symbol Device:C_Small
- added C4, C5: 15p, Capacitor_SMD:C_0402_1005Metric, symbol Device:C_Small
- added D2: ERR, LED_SMD:LED_0603_1608Metric_Pad1.05x0.95mm_HandSolder, symbol Device:LED
- added D3: 1N4148WS, Diode_SMD:D_SOD-323, symbol Diode:1N4148WS
- added FID1, FID2, FID3, FID4: Fiducial, Fiducial:Fiducial_1.5mm_Mask3mm, symbol Mechanical:Fiducial
- added H1, H2, H3, H4: MOUNT, MountingHole:MountingHole_3.2mm_M3_Pad_Via, symbol Mechanical:MountingHole_Pad_MP
- added H5: TRIPOD, MountingHole:MountingHole_8.4mm_M8_Pad_Via, symbol Mechanical:MountingHole_Pad_MP
- added J1: SERIAL_DEBUG, Connector_JST:JST_SH_SM03B-SRSS-TB_1x03-1MP_P1.00mm_Horizontal, symbol Connector_Generic_MountingPin:Conn_01x03_MountingPin
- added J2: SWD, Connector_JST:JST_SH_SM03B-SRSS-TB_1x03-1MP_P1.00mm_Horizontal, symbol Connector_Generic_MountingPin:Conn_01x03_MountingPin
- added J3: USB, Connector_USB:USB_C_Receptacle_G-Switch_GT-USB-7010ASV, symbol Connector:USB_C_Receptacle_USB2.0_14P
- added L1: 3.3uH, Inductor_SMD:L_0805_2012Metric, symbol Device:L_Small
- added Q1: AO3401A, Package_TO_SOT_SMD:SOT-23, symbol Transistor_FET:AO3401A
- added Q2: 2N7002, PCM_Package_TO_SOT_SMD_AKL:SOT-23, symbol PCM_Transistor_MOSFET_AKL:2N7002
- added R11, R8: 10k, Resistor_SMD:R_0402_1005Metric, symbol Device:R
- added R12: 270, Resistor_SMD:R_0402_1005Metric, symbol Device:R
- added R15, R9: 1k, Resistor_SMD:R_0402_1005Metric, symbol Device:R
- added R16: 330, Resistor_SMD:R_0603_1608Metric, symbol Device:R
- added R17, R18, R19: 4.7k, Resistor_SMD:R_0805_2012Metric, symbol Device:R
- added R21: 390k, Resistor_SMD:R_0805_2012Metric, symbol Device:R
- added SW3: DOWN, Button_Switch_SMD:SW_SPST_EVPBF, symbol Switch:SW_SPST
- added SW4: UP, Button_Switch_SMD:SW_SPST_EVPBF, symbol Switch:SW_SPST
- added SW5: CART_TYPE_SELECT, gbpunk:SW_DPDT_CK_JS202011JCQN, symbol Switch:SW_Slide_DPDT
- added SW6: A, Button_Switch_SMD:SW_SPST_EVPBF, symbol Switch:SW_SPST
- added SW7: B, Button_Switch_SMD:SW_SPST_EVPBF, symbol Switch:SW_SPST
- added TP3: RUN_TP, TestPoint:TestPoint_2Pads_Pitch2.54mm_Drill0.8mm, symbol Connector:TestPoint_2Pole
- added TP4: USB_TP, TestPoint:TestPoint_2Pads_Pitch2.54mm_Drill0.8mm, symbol Connector:TestPoint_2Pole
- added U3: RP2350B, Package_DFN_QFN:QFN-80-1EP_10x10mm_P0.4mm_EP3.4x3.4mm, symbol MCU_RaspberryPi:RP2350B
- added U7: SSD1306, gbpunk:SSD1306, symbol tmg_2025_hardware:SSD1306
- added Y1: 12MHz, Crystal:Crystal_SMD_3225-4Pin_3.2x2.5mm, symbol Device:Crystal_GND24
- C10, C13, C14, C15, C16, C17, C18, C19, C20: footprint Capacitor_SMD:C_0402_1005Metric_Pad0.74x0.62mm_HandSolder -> Capacitor_SMD:C_0402_1005Metric
- C11: value 1uF -> 4.7uF; footprint Capacitor_SMD:C_0805_2012Metric_Pad1.18x1.45mm_HandSolder -> Capacitor_SMD:C_0805_2012Metric
- C12: value 1uF -> 100nF; footprint Capacitor_SMD:C_0805_2012Metric_Pad1.18x1.45mm_HandSolder -> Capacitor_SMD:C_0402_1005Metric
- C25: renamed from C22; footprint Capacitor_SMD:C_0402_1005Metric_Pad0.74x0.62mm_HandSolder -> Capacitor_SMD:C_0402_1005Metric
- C6: renamed from C21; footprint Capacitor_SMD:C_1206_3216Metric_Pad1.33x1.80mm_HandSolder -> Capacitor_SMD:C_0603_1608Metric
- C7: renamed from C23; footprint Capacitor_SMD:C_1206_3216Metric_Pad1.33x1.80mm_HandSolder -> Capacitor_SMD:C_0603_1608Metric
- C8: value 27pF -> 2.2uF; footprint Capacitor_SMD:C_0402_1005Metric_Pad0.74x0.62mm_HandSolder -> Capacitor_SMD:C_0603_1608Metric_Pad1.08x0.95mm_HandSolder
- C9: value 100nF -> 2.2uF; footprint Capacitor_SMD:C_0402_1005Metric_Pad0.74x0.62mm_HandSolder -> Capacitor_SMD:C_0603_1608Metric_Pad1.08x0.95mm_HandSolder
- J4: renamed from J1; footprint gbpunk:gbpunk_aliexpress_gb_connector -> Connector_PinSocket_2.54mm:PinSocket_1x32_P2.54mm_Vertical
- R1: value 1k -> 33; footprint Resistor_SMD:R_0603_1608Metric_Pad0.98x0.95mm_HandSolder -> Resistor_SMD:R_0603_1608Metric
- R10: renamed from R14; footprint Resistor_SMD:R_0603_1608Metric_Pad0.98x0.95mm_HandSolder -> Resistor_SMD:R_0603_1608Metric
- R13: value 1k -> 10k; footprint Resistor_SMD:R_0603_1608Metric_Pad0.98x0.95mm_HandSolder -> Resistor_SMD:R_0402_1005Metric
- R2: renamed from R18; value 56k -> 5.1k; footprint Resistor_SMD:R_0402_1005Metric_Pad0.72x0.64mm_HandSolder -> Resistor_SMD:R_0402_1005Metric
- R20: renamed from R19; footprint Resistor_SMD:R_0402_1005Metric_Pad0.72x0.64mm_HandSolder -> Resistor_SMD:R_0402_1005Metric
- R3: renamed from R15; value 56k -> 5.1k; footprint Resistor_SMD:R_0402_1005Metric_Pad0.72x0.64mm_HandSolder -> Resistor_SMD:R_0402_1005Metric
- R4: renamed from R8; footprint Resistor_SMD:R_0402_1005Metric_Pad0.72x0.64mm_HandSolder -> Resistor_SMD:R_0402_1005Metric
- R5: renamed from R12; footprint Resistor_SMD:R_0603_1608Metric_Pad0.98x0.95mm_HandSolder -> Resistor_SMD:R_0603_1608Metric
- R6: renamed from R11; footprint Resistor_SMD:R_0603_1608Metric_Pad0.98x0.95mm_HandSolder -> Resistor_SMD:R_0603_1608Metric
- R7: renamed from R9; footprint Resistor_SMD:R_0402_1005Metric_Pad0.72x0.64mm_HandSolder -> Resistor_SMD:R_0402_1005Metric
- TP5: value 5V0_TP -> VBUS_TP
- U8: renamed from U3; footprint Package_SO:SOIC-8_5.23x5.23mm_P1.27mm -> Package_SO:SOIC-8_5.3x5.3mm_P1.27mm
- renumbered SW7 to SW1, SW9 to SW2, TP3 to TP2, U2 to U1, U5 to U2, U6 to U4, U7 to U5, U4 to U6
Connections:
- net +1V1: now also C12.1, U3.10 (DVDD), U3.32 (DVDD), U3.51 (DVDD); no longer C9.1
- net +3.3V: now also R1.1, C2.1, C21.1, C22.1, C23.1, D2.2 (A), D3.1 (K), R17.2, R18.2, R19.1, SW5.1 (A), SW5.6 (C), U3.15 (IOVDD), U3.24 (IOVDD), U3.29 (IOVDD), U3.41 (IOVDD), U3.5 (IOVDD), U3.50 (IOVDD), U3.59 (ADC_AVDD), U3.60 (IOVDD), U3.64 (VREG_VIN), U3.68 (USB_OTP_VDD), U3.69 (QSPI_IOVDD), U3.76 (IOVDD), U7.11 (BS1), U7.6 (VBAT), U7.9 (VDD); no longer C12.1
- net A0: now also U4.10 (A8); no longer U5.6 (A4)
- net A0_L: now also U4.14 (B8), U3.25 (GPIO24); no longer U5.18 (B4)
- net A1: now also U4.9 (A7); no longer U5.5 (A3)
- net A10: now also U2.8 (A6); no longer U4.4 (A2)
- net A10_L: now also U2.16 (B6), U3.13 (GPIO14); no longer U4.20 (B2)
- net A11: now also U2.7 (A5); no longer U4.3 (A1)
- net A11_L: now also U2.17 (B5), U3.12 (GPIO13); no longer U4.21 (B1)
- net A12: now also U2.6 (A4); no longer U2.10 (A8)
- net A12_L: now also U2.18 (B4), U3.11 (GPIO12); no longer U2.14 (B8)
- net A13: now also U2.5 (A3); no longer U2.9 (A7)
- net A13_L: now also U2.19 (B3), U3.9 (GPIO11); no longer U2.15 (B7)
- net A14: now also U2.4 (A2); no longer U2.8 (A6)
- net A14_L: now also U2.20 (B2), U3.8 (GPIO10); no longer U2.16 (B6)
- net A15: now also U2.3 (A1); no longer U2.7 (A5)
- net A15_L: now also U2.21 (B1), U3.7 (GPIO9); no longer U2.17 (B5)
- net A1_L: now also U4.15 (B7), U3.23 (GPIO23); no longer U5.19 (B3)
- net A2: now also U4.8 (A6); no longer U5.4 (A2)
- net A2_L: now also U4.16 (B6), U3.22 (GPIO22); no longer U5.20 (B2)
- net A3: now also U4.7 (A5); no longer U5.3 (A1)
- net A3_L: now also U4.17 (B5), U3.21 (GPIO21); no longer U5.21 (B1)
- net A4: now also U4.6 (A4); no longer U4.10 (A8)
- net A4_L: now also U4.18 (B4), U3.20 (GPIO20); no longer U4.14 (B8)
- net A5: now also U4.5 (A3); no longer U4.9 (A7)
- net A5_L: now also U4.19 (B3), U3.19 (GPIO19); no longer U4.15 (B7)
- net A6: now also U4.4 (A2); no longer U4.8 (A6)
- net A6_L: now also U4.20 (B2), U3.18 (GPIO18); no longer U4.16 (B6)
- net A7: now also U4.3 (A1); no longer U4.7 (A5)
- net A7_L: now also U4.21 (B1), U3.17 (GPIO17); no longer U4.17 (B5)
- net A8: now also U2.10 (A8); no longer U4.6 (A4)
- net A8_L: now also U2.14 (B8), U3.16 (GPIO16); no longer U4.18 (B4)
- net A9: now also U2.9 (A7); no longer U4.5 (A3)
- net A9_L: now also U2.15 (B7), U3.14 (GPIO15); no longer U4.19 (B3)
- net CLK: now also U5.6 (A4); no longer U5.10 (A8)
- net CLK_L: now also U5.18 (B4), U3.36 (GPIO28); no longer U5.14 (B8)
- net D0_L: now also U3.4 (GPIO7)
- net D1_L: now also U3.3 (GPIO6)
- net D2_L: now also U3.2 (GPIO5)
- net D3_L: now also U3.1 (GPIO4)
- net D4_L: now also U3.80 (GPIO3)
- net D5_L: now also U3.79 (GPIO2)
- net D6_L: now also U3.78 (GPIO1)
- net D7_L: now also U3.77 (GPIO0)
- net GND: now also R13.1, R2.1, U5.10 (A8), U5.14 (B8), U5.15 (B7), U5.9 (A7), C1.2, C2.2, C21.2, C22.2, C23.2, C24.1, C26.2, C27.2, C3.2, C4.1, C5.1, H1.MP, H2.MP, H3.MP, H4.MP, H5.MP, J1.2 (Pin_2), J1.MP (MountPin), J2.2 (Pin_2), J2.MP (MountPin), J3.A1 (GND), J3.A12 (GND), J3.B1 (GND), J3.B12 (GND), J3.S1 (SHIELD), Q2.2 (S), R11.1, R21.1, SW3.1 (A), SW4.1 (A), SW5.4 (A), SW6.1 (A), SW7.1 (A), TP3.1, U3.62 (VREG_PGND), U3.81 (GND), U7.1 (NC(GND)), U7.10 (BS0), U7.12 (BS2), U7.13 (/CS), U7.15 (DC/I2C_SAO), U7.16 (R/W), U7.17 (E/RD), U7.21 (D3), U7.22 (D4), U7.23 (D5), U7.24 (D6), U7.25 (D7), U7.29 (VLSS), U7.30 (NC(GND)), U7.8 (VSS), Y1.2, Y1.4; no longer C8.2, C9.2, R13.2, R2.2, U2.19 (B3), U2.20 (B2), U2.21 (B1), U2.3 (A1), U2.4 (A2), U2.5 (A3)
- net QSPI_CLK: now also U3.71 (QSPI_SCLK)
- net QSPI_D0: now also U3.72 (QSPI_SD0)
- net QSPI_D1: now also U3.74 (QSPI_SD1)
- net QSPI_D2: now also U3.73 (QSPI_SD2)
- net QSPI_D3: now also U3.70 (QSPI_SD3)
- net RST: now also U5.7 (A5); no longer U2.6 (A4)
- net RST_L: now also U5.17 (B5), U3.37 (GPIO29); no longer U2.18 (B4)
- net SWCLK: now also J2.1 (Pin_1), U3.33 (SWCLK)
- net SWDIO: now also J2.3 (Pin_3), U3.34 (SWDIO)
- net USB_DM: now also J3.A7 (D-), J3.B7 (D-), TP4.2
- net USB_DP: now also J3.A6 (D+), J3.B6 (D+), TP4.1
- net VBUS: now also C6.1, F1.1, TP5.1, U6.3 (VI), SW5.3 (C); no longer F1.2
- net ~{CS_L}: now also U5.21 (B1), U3.26 (GPIO25); no longer U5.17 (B5)
- net ~{CS}: now also U5.3 (A1), R15.2; no longer U5.7 (A5)
- net ~{QSPI_CS}: now also U3.75 (~{QSPI_SS})
- net ~{RD_L}: now also U5.20 (B2), U3.27 (GPIO26); no longer U5.16 (B6)
- net ~{RD}: now also U5.4 (A2); no longer U5.8 (A6)
- net ~{WR_L}: now also U5.19 (B3), U3.28 (GPIO27); no longer U5.15 (B7)
- net ~{WR}: now also U5.5 (A3); no longer U5.9 (A7)
- net at C8.1: now also U7.2 (C2P)
- net at R6.2: now also U3.67 (USB_DP)
- net at R5.2: now also U3.66 (USB_DM)
- net at R10.2: now also U3.6 (GPIO8)
- net ABUS1_OE: now reaches U2.22 (~{OE})
- net ABUS1_OE: now also U3.44 (GPIO35)
- net DBUS_DIR: now reaches U1.2 (DIR)
- net DBUS_DIR: now also U3.47 (GPIO38)
- net at R3.1: now also J3.B5 (CC2)
- net IRQ: now reaches J4.31 (Pin_31)
- net IRQ: now also U5.8 (A6)
- net CTLBUS_OE: now reaches U5.22 (~{OE})
- net CTLBUS_OE: now also U3.39 (GPIO31); no longer R13.1
- net CTLBUS_DIR: now reaches U5.2 (DIR)
- net CTLBUS_DIR: now also U3.40 (GPIO32); no longer R1.1
- net VREG_AVDD: now reaches R1.2
- net VREG_AVDD: now also C1.1, U3.61 (VREG_AVDD)
- net ABUS0_OE: now reaches U4.22 (~{OE})
- net ABUS0_OE: now also U3.42 (GPIO33)
- net ABUS0_DIR: now reaches U4.2 (DIR)
- net ABUS0_DIR: now also U3.43 (GPIO34)
- net DBUS_OE: now reaches U1.22 (~{OE})
- net DBUS_OE: now also U3.46 (GPIO37)
- net ABUS1_DIR: now reaches U2.2 (DIR)
- net ABUS1_DIR: now also U3.45 (GPIO36)
- net +5V renamed GB_POWER_SW
- net GB_POWER_SW: now also Q1.2 (S), R11.2, R15.1; no longer C6.1, F1.1, TP5.1, U6.3 (VI)
- net RUN: no longer names the net of R4.2, SW1.2 (B)
- net RUN: now also TP3.2, U3.35 (RUN)
- new net: F1.2, J3.A4 (VBUS), J3.A9 (VBUS), J3.B4 (VBUS), J3.B9 (VBUS)
- new net: J3.A5 (CC1), R2.2
- new net: C9.1, U7.4 (C1P)
- new net: C9.2, U7.5 (C1N)
- new net: C5.2, R9.1, Y1.3
- new net: Q1.3 (D), R8.2, SW5.2 (B)
- new net: R21.2, U7.26 (IREF)
- new net: C4.2, U3.30 (XIN), Y1.1
- new net: R9.2, U3.31 (XOUT)
- new net: R16.2, U3.58 (GPIO47/ADC7)
- new net: C24.2, D3.2 (A), R19.2, U7.14 (/RES)
- new net: Q2.1 (G), R12.1, R13.2
- new net: Q1.1 (G), Q2.3 (D), R8.1
- new net: C8.2, U7.3 (C2N)
- new net: D2.1 (K), R16.1
- new net: C26.1, U7.27 (VCOMH)
- new net: C27.1, U7.28 (VCC)
- new net 1V1_INTERNAL: C3.1, L1.1, U3.65 (VREG_FB)
- new net A: SW6.2 (B), U3.54 (GPIO43/ADC3)
- new net B: SW7.2 (B), U3.57 (GPIO46/ADC6)
- new net CART_TYPE_SELECT: SW5.5 (B), U3.48 (GPIO39)
- new net DEBUG_RX: J1.1 (Pin_1)
- new net DEBUG_TX: J1.3 (Pin_3)
- new net DOWN: SW3.2 (B), U3.52 (GPIO41/ADC1)
- new net GB_POWER_EN: R12.2, U3.49 (GPIO40/ADC0)
- new net IRQ_L: U3.38 (GPIO30), U5.16 (B6)
- new net SCREEN_SCL: R18.1, U3.56 (GPIO45/ADC5), U7.18 (D0/SPI_SCLK/I2C_SCK)
- new net SCREEN_SDA: R17.1, U3.55 (GPIO44/ADC4), U7.19 (D1/SPI_SDIN/I2C_SDA), U7.20 (D2/I2C_SDA)
- new net UP: SW4.2 (B), U3.53 (GPIO42/ADC2)
- new net VREG_LX: L1.2, U3.63 (VREG_LX)
- no-connect marks 14 -> 1
Other:
- note added: "Bulk Decoupling (Keep close to Power Pins)"
- note added: "RP2350 Main Micro"
- note removed: "RP2040 Main Micro"
- company: (none) -> Kay Barkbark
- title: (none) -> gbpunk
- moved on the sheet: C25, C6, C7, D1, F1, J4, R10, R2, R20, R3, R4, R5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

Commit message: ready to start version 2.0. picking this project back up, technology and I have both progresses
Parts:
- removed H1, H2, H3, H4: MOUNT, MountingHole:MountingHole_3.2mm_M3_Pad_Via, symbol Mechanical:MountingHole_Pad_MP
- removed H5: TRIPOD, MountingHole:MountingHole_8.4mm_M8_Pad_Via, symbol Mechanical:MountingHole_Pad_MP
- added H1, H2, H3, H4: MOUNT, MountingHole:MountingHole_3.2mm_M3_Pad_Via, symbol Mechanical:MountingHole_Pad
- added H5: TRIPOD, MountingHole:MountingHole_8.4mm_M8_Pad_Via, symbol Mechanical:MountingHole_Pad
- R12: value 270 -> 330
Connections:
- net GND: now also H1.1, H2.1, H3.1, H4.1, H5.1
