File: hardware/tht_gb_adapter/tht_gb_adapter.kicad_pcb (KiCad board)
At the start: 2 copper layers, 83.8 x 40.5 mm, 2 parts, among them J1 CART, J2 THT_ADAPTER

Commit message: ready to start version 2.0. picking this project back up, technology and I have both progresses
Parts:
- added REF**: boykisser_10mm, pawprint_kicad_art:boykisser_10mm, F.Cu at (143.1, 76.1)
